File: design_files/ASL2112.sch (EAGLE design)
At the start: 13 parts, among them J1 47346-0001, J2 SM02B-SRSS-TB(LF)(SN), J3 PIN_1X.1"1, J4 PIN_1X.1"1, U1 MCP73831

Commit message: update format
Parts:
- removed D2: GREEN, tinycircuits:AS-ITM-00038
- added R4, R5: 0.0, tinycircuits:AS-ITM-00076
- D1: value RED -> AMBER; device tinycircuits:AS-ITM-00057 -> tinycircuits:AS-ITM-00058; PARTNO AS-ITM-00057 -> AS-ITM-00058; VALUE RED -> AMBER
- R2: device tinycircuits:AS-ITM-00003 -> tinycircuits:AS-ITM-00315; PARTNO AS-ITM-00003 -> AS-ITM-00315; VALUE 1.00K -> 2K
Connections:
- new net N$4: R2.1, R4.2
- new net N$7: R3.1, R5.2
- net GND: now also R2.2, R3.2; no longer D2.C, R2.1, R3.1
- net N$2: no longer D2.A
- net N$3: now also R4.1, R5.1; no longer R2.2, R3.2
Other:
- note added: "2"
- note added: "Hand Populated: -"
- note added: "Hand Soldered: -"
- note added: "Non Populated: R4"
- note added: "Notes: -"
- note added: "R4: 0.5A setting, not populated by default"
- note added: "R5: 0.1A setting, populated by default"
- note added: "Variant: Standard"
- note removed: "1"
- note removed: "D1 charge active indicator populated by default"
- note removed: "D1/D2 optionally populated!"
- note removed: "D2 charge complete indicator non-populated by default"
- note removed: "R2: 0.5A setting, not populated by default"
- note removed: "R3: 0.1A setting, populated by default"
- moved on the sheet: C1, C2, C3, D1, J1, J2, J3, J4, R1, R2, R3, U1
